File: hs100b-eval.kicad_pcb (KiCad board)
At the start: 2 copper layers, 60 x 50 mm, 42 parts, among them IC1 HS-100B, J1 USB_B_Micro, J2 SPKR, J20 RADIO_DATA, J3 MIC, SW1 MUTE_REC, SW2 MUTE_PLAY, SW3 VOL_DN, SW4 VOL_UP, SW5 SW_DIP_x03

Commit message: Add OSHW logo
Parts:
- added LOGO1: Logo_Open_Hardware_Small, Symbol:OSHW-Logo2_9.8x8mm_SilkScreen, B.Cu at (170.0, 100.0)
