File: hs100b-eval.sch (KiCad schematic (older format))
At the start: 43 parts, among them IC1 HS-100B, J1 SPKR, J2 MIC, J3 RADIO_DATA, SW1 MUTE_REC, SW2 MUTE_PLAY, SW3 VOL_DN, SW4 VOL_UP, SW5 SW_DIP_x03

Commit message: Renumber components
Parts:
- removed D3: PWR_DN, LED_SMD:LED_0603_1608Metric, symbol Device:LED_ALT
- removed R7: 330Ω, Resistor_SMD:R_1210_3225Metric, symbol Device:R_Small_US
- added R1: 0Ω, Resistor_SMD:R_1210_3225Metric, symbol Device:R_Small_US
- L1, L2: value L -> Ferrite_Bead
- renumbered C10 to C1, C50 to C10, C51 to C11, C15 to C12, C11 to C13, C1 to C21, C9 to C3, C8 to C4, C7 to C5, C4 to C7, C3 to C8, C14 to C9, JP2 to J1, J1 to J2, J3 to J20, J2 to J3, R5 to R2, R3 to R21, R6 to R22, R4 to R3, R2 to R4, R1 to R5, R10 to R6, R13 to R7, R11 to R8, R12 to R9
Connections:
- net VBUS: now also R1.2; no longer IC1.35 (DVDD)
- net AVDD2: now reaches C5.1, C6.1, IC1.34 (AVDD_2), R3.1
- net AVDD1: now reaches C3.1, C4.1, IC1.29 (AVDD_1), R2.1
- new net DVDD: IC1.35 (DVDD), R1.1
Other:
- moved on the sheet: C1, C10, C11, C12, C13, C3, C4, C5, C6, C7, C8, C9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

Commit message: Swap Diptronics switches for smaller Wurth one
Parts:
- SW5: footprint Diptronics:DMR -> Wurth:416131160803; Price 1.72 -> 3.31; Vendor Part # 113-DMR03V -> 710-416131160803
Changed lines of the file:
@@
 Title "HS100B Evaluation Board"
 Date "2021-04-21"
-Rev "3"
+Rev "4"
 Comp "Chris Keller"
 Comment1 "Licensed under Creative Commons CC-BY-4.0"
@@
 F 0 "SW5" V 2050 5170 50  0000 R CNN
 F 1 "SW_DIP_x03" V 2005 5170 50  0001 R CNN
-F 2 "Diptronics:DMR" H 2050 5300 50  0001 C CNN
-F 3 "https://www.mouser.com/datasheet/2/910/374_DM-1544377.pdf" H 2050 5300 50  0001 C CNN
-F 4 "1.72" H 2050 5300 50  0001 C CNN "Price"
+F 2 "Wurth:416131160803" H 2050 5300 50  0001 C CNN
+F 3 "https://www.mouser.com/datasheet/2/445/416131160803-1717247.pdf" H 2050 5300 50  0001 C CNN
+F 4 "3.31" H 2050 5300 50  0001 C CNN "Price"
 F 5 "Mouser" H 2050 5300 50  0001 C CNN "Vendor"
-F 6 "113-DMR03V" H 2050 5300 50  0001 C CNN "Vendor Part #"
+F 6 "710-416131160803" H 2050 5300 50  0001 C CNN "Vendor Part #"
 	1    2050 5300
 	0    -1   -1   0

Commit message: Fix R and L channels
Connections:
- net at C10.1: now also IC1.30 (LOL); no longer IC1.32 (LOR)
- net at C11.1: now also IC1.32 (LOR); no longer IC1.30 (LOL)
Other:
- moved on the sheet: C10, C11
Changed lines of the file:
@@
 L Device:CP C10
 U 1 1 606A39C6
-P 6550 4600
-F 0 "C10" V 6805 4600 50  0000 C CNN
-F 1 "470μF" V 6714 4600 50  0000 C CNN
-F 2 "Vishay:CAPPM7343X430N" H 6588 4450 50  0001 C CNN
-F 3 "https://www.mouser.com/datasheet/2/427/293d-1763499.pdf" H 6550 4600 50  0001 C CNN
-F 4 "1.3" H 6805 4700 50  0001 C CNN "Price"
-F 5 "74-293D477X9010E2TE3" V 6550 4600 50  0001 C CNN "Vendor Part #"
-F 6 "Mouser" H 6805 4700 50  0001 C CNN "Vendor"
-	1    6550 4600
-	0    -1   -1   0
-$EndComp
-$Comp
-L Device:CP C11
-U 1 1 606A46F9
-P 6850 4700
-F 0 "C11" V 7100 4700 50  0000 C CNN
-F 1 "470μF" V 7000 4700 50  0000 C CNN
-F 2 "Vishay:CAPPM7343X430N" H 6888 4550 50  0001 C CNN
-F 3 "https://www.mouser.com/datasheet/2/427/293d-1763499.pdf" H 6850 4700 50  0001 C CNN
-F 4 "1.3" H 7100 4800 50  0001 C CNN "Price"
-F 5 "74-293D477X9010E2TE3" V 6850 4700 50  0001 C CNN "Vendor Part #"
-F 6 "Mouser" H 7100 4800 50  0001 C CNN "Vendor"
-	1    6850 4700
+P 6550 4700
+F 0 "C10" V 6805 4700 50  0000 C CNN
+F 1 "470μF" V 6714 4700 50  0000 C CNN
+F 2 "Vishay:CAPPM7343X430N" H 6588 4550 50  0001 C CNN
+F 3 "https://www.mouser.com/datasheet/2/427/293d-1763499.pdf" H 6550 4700 50  0001 C CNN
+F 4 "1.3" H 6805 4800 50  0001 C CNN "Price"
+F 5 "74-293D477X9010E2TE3" V 6550 4700 50  0001 C CNN "Vendor Part #"
+F 6 "Mouser" H 6805 4800 50  0001 C CNN "Vendor"
+	1    6550 4700
 	0    -1   -1   0
 $EndComp
@@
 Text Label 7400 5200 0    50   ~ 0
 MIC_BIAS
-Text Label 7400 4600 0    50   ~ 0
+Text Label 7400 4700 0    50   ~ 0
 AUDIO_L
-Text Label 7400 4700 0    50   ~ 0
-AUDIO_R
 Text Label 8650 4350 2    50   ~ 0
 MIC_IN
@@
 	4300 1200 4550 1200
 Wire Wire Line
-	5700 4600 6400 4600
-Wire Wire Line
-	5700 4700 6700 4700
+	5700 4700 6400 4700
 Wire Wire Line
 	8650 3950 8900 3950
@@
 	8900 4550 8800 4550
 Wire Wire Line
-	6700 4600 7400 4600
-Wire Wire Line
-	7000 4700 7400 4700
+	6700 4700 7400 4700
 Wire Wire Line
 	7150 5100 7400 5100
@@
 Text Label 5700 4050 0    50   ~ 0
 AVDD2
+Wire Wire Line
+	7000 4600 7400 4600
+Wire Wire Line
+	5700 4600 6700 4600
+Text Label 7400 4600 0    50   ~ 0
+AUDIO_R
+$Comp
+L Device:CP C11
+U 1 1 606A46F9
+P 6850 4600
+F 0 "C11" V 7100 4600 50  0000 C CNN
+F 1 "470μF" V 7000 4600 50  0000 C CNN
+F 2 "Vishay:CAPPM7343X430N" H 6888 4450 50  0001 C CNN
+F 3 "https://www.mouser.com/datasheet/2/427/293d-1763499.pdf" H 6850 4600 50  0001 C CNN
+F 4 "1.3" H 7100 4700 50  0001 C CNN "Price"
+F 5 "74-293D477X9010E2TE3" V 6850 4600 50  0001 C CNN "Vendor Part #"
+F 6 "Mouser" H 7100 4700 50  0001 C CNN "Vendor"
+	1    6850 4600
+	0    -1   -1   0
+$EndComp
 $EndSCHEMATC

Commit message: Add OSHW logo
Parts:
- added LOGO1: Logo_Open_Hardware_Small, Symbol:OSHW-Logo2_9.8x8mm_SilkScreen, symbol Graphic:Logo_Open_Hardware_Small
Changed lines of the file:
@@
 	0    -1   -1   0
 $EndComp
+$Comp
+L Graphic:Logo_Open_Hardware_Small LOGO1
+U 1 1 6083E287
+P 10900 6850
+F 0 "LOGO1" H 10900 7125 50  0001 C CNN
+F 1 "Logo_Open_Hardware_Small" H 10900 6625 50  0001 C CNN
+F 2 "Symbol:OSHW-Logo2_9.8x8mm_SilkScreen" H 10900 6850 50  0001 C CNN
+F 3 "~" H 10900 6850 50  0001 C CNN
+	1    10900 6850
+	1    0    0    -1
+$EndComp
 $EndSCHEMATC
